Commit message: trying to launch navigation

File: src/acds_description/urdf/robot.urdf.xacro (robot description, xacro)
@@ -2,10 +2,11 @@
 <robot xmlns:xacro="http://www.ros.org/wiki/xacro" name="acds_robot">
   <!-- PROPERTIES -->
-  <xacro:property name="wheel_radius" value="0.035"/>
+  <xacro:property name="wheel_radius" value="0.0325"/>
   <xacro:property name="wheel_width" value="0.025"/>
   <xacro:property name="wheelbase" value="0.26"/>
-  <xacro:property name="track_width" value="0.18"/>
-  <xacro:property name="chassis_length" value="0.30"/>
-  <xacro:property name="chassis_width" value="0.20"/>
+  <xacro:property name="track_width" value="0.12"/>
+  <xacro:property name="chassis_length" value="0.26"/>
+  <xacro:property name="chassis_width" value="0.09
+  "/>
   <xacro:property name="chassis_height" value="0.10"/>
   <!-- BASE_FOOTPRINT (Ground projection) -->
